File: src/1.0/RJ45-LED-Breakout.brd (EAGLE design)
At the start: 16.5 x 27.9 mm, 5 parts, among them J1 RJ45-RJHSE-5481

Commit message: Switching to develop branch.
Other:
- board size 16.5 x 27.9 mm -> 16.5 x 29.2 mm
Changed lines of the file:
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@@
 <plain>
 <wire x1="0" y1="0" x2="16.49" y2="0" width="0" layer="20"/>
-<wire x1="16.49" y1="0" x2="16.49" y2="27.864" width="0" layer="20"/>
-<wire x1="16.49" y1="27.864" x2="0" y2="27.864" width="0" layer="20"/>
-<wire x1="0" y1="27.864" x2="0" y2="0" width="0" layer="20"/>
+<wire x1="16.49" y1="0" x2="16.51" y2="29.21" width="0" layer="20"/>
+<wire x1="16.51" y1="29.21" x2="0" y2="29.21" width="0" layer="20"/>
+<wire x1="0" y1="29.21" x2="0" y2="0" width="0" layer="20"/>
 </plain>
 <attributes>
