File: src/1.0/RJ45-LED-Breakout.brd (EAGLE design)
At the start: 16.5 x 30.5 mm, 7 parts, among them J1 RJ45-RJHSE-5481, J2 M06SQ1, J3 M06SQ1

Commit message: Almost ready for release. Need to create BOM and review all connections. Also look over schematic and possibly clean things up if necessary.
Parts:
- added LOGO1: OSHW-LOGOM, SparkFun-Aesthetics:OSHW-LOGO-M
Connections:
- net N$3: now also J1.7; no longer J1.8
- net N$4: now also J1.8; no longer J1.7
Routing:
- net N$4: track 12.0 -> 8.72 mm
- net N$3: track 8.93 -> 11.1 mm
Other:
- board text added: "Breakout"
Changed lines of the file:
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@@
 <text x="13.462" y="27.178" size="1.524" layer="22" font="vector" ratio="12" rot="MR0">RJ45-LED</text>
 <text x="3.556" y="16.51" size="1.524" layer="22" font="vector" ratio="12" rot="MR270">v1.0</text>
+<text x="13.208" y="-0.508" size="1.524" layer="22" font="vector" ratio="12" rot="MR0">Breakout</text>
 </plain>
 <attributes>
@@
 <elements>
 <element name="J1" library="LoganSmith-Connectors" package="RJ45-RJHSE" value="RJ45-RJHSE-5481" x="7.112" y="13.97" smashed="yes" rot="R270">
-<attribute name="LED1_COLOR" value="GRN" x="8.89" y="8.128" size="1.016" layer="51" font="vector" ratio="12" rot="R270" align="bottom-center"/>
-<attribute name="LED2_COLOR" value="YEL" x="8.89" y="19.685" size="1.016" layer="51" font="vector" ratio="12" rot="R270" align="bottom-center"/>
+<attribute name="LED1_COLOR" value="GRN" x="14.732" y="5.08" size="1.016" layer="21" font="vector" ratio="12" rot="R180" align="bottom-center"/>
+<attribute name="LED2_COLOR" value="YEL" x="11.811" y="5.08" size="1.016" layer="21" font="vector" ratio="12" rot="R180" align="bottom-center"/>
 <attribute name="VALUE" x="2.286" y="13.97" size="1.016" layer="27" font="vector" ratio="12" rot="R270" align="bottom-center"/>
 </element>
@@
 <attribute name="VALUE" x="0.254" y="4.445" size="1" layer="27" font="vector" ratio="12"/>
 </element>
+<element name="LOGO1" library="SparkFun-Aesthetics" package="OSHW-LOGO-M" value="OSHW-LOGOM" x="11.176" y="13.97" rot="MR270"/>
 </elements>
 <signals>
@@
 <signal name="N$3">
 <contactref element="J2" pad="3"/>
-<contactref element="J1" pad="8"/>
-<wire x1="7.112" y1="17.526" x2="8.128" y2="18.542" width="0.254" layer="1"/>
-<wire x1="8.128" y1="18.542" x2="8.128" y2="22.86" width="0.254" layer="1"/>
-<wire x1="8.128" y1="22.86" x2="6.604" y2="24.384" width="0.254" layer="1"/>
-<wire x1="6.604" y1="24.384" x2="6.604" y2="25.4" width="0.254" layer="1"/>
+<contactref element="J1" pad="7"/>
+<wire x1="5.334" y1="16.51" x2="5.334" y2="17.526" width="0.254" layer="1"/>
+<wire x1="5.334" y1="17.526" x2="8.636" y2="20.828" width="0.254" layer="1"/>
+<wire x1="8.636" y1="20.828" x2="8.636" y2="23.368" width="0.254" layer="1"/>
+<wire x1="8.636" y1="23.368" x2="6.604" y2="25.4" width="0.254" layer="1"/>
 </signal>
 <signal name="N$4">
 <contactref element="J2" pad="4"/>
-<contactref element="J1" pad="7"/>
-<wire x1="5.334" y1="16.51" x2="7.874" y2="16.51" width="0.254" layer="1"/>
-<wire x1="7.874" y1="16.51" x2="8.636" y2="17.272" width="0.254" layer="1"/>
-<wire x1="8.636" y1="17.272" x2="8.636" y2="22.86" width="0.254" layer="1"/>
-<wire x1="8.636" y1="22.86" x2="9.144" y2="23.368" width="0.254" layer="1"/>
-<wire x1="9.144" y1="23.368" x2="9.144" y2="25.4" width="0.254" layer="1"/>
+<contactref element="J1" pad="8"/>
+<wire x1="7.112" y1="17.526" x2="9.144" y2="19.558" width="0.254" layer="1"/>
+<wire x1="9.144" y1="19.558" x2="9.144" y2="25.4" width="0.254" layer="1"/>
 </signal>
 </signals>

Commit message: Board has been ordered. Updated README, finalized board layout and silk. Need to create BOM and release 1.0.
Parts:
- J2, J3: value M06SQ1 -> (none)
- moved J2 0.25 mm to (1.78, 25.4)
- moved J3 0.25 mm to (1.78, 2.54)
- moved LOGO1 0.25 mm to (10.9, 14.0), turned to 90 degrees
- moved SJ1 0.13 mm to (5.71, 8.38)
- moved SJ2 0.13 mm to (5.71, 19.6)
Other:
- board text added: "RJHSE-548x"
Changed lines of the file:
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@@
 <text x="3.556" y="16.51" size="1.524" layer="22" font="vector" ratio="12" rot="MR270">v1.0</text>
 <text x="13.208" y="-0.508" size="1.524" layer="22" font="vector" ratio="12" rot="MR0">Breakout</text>
+<text x="10.16" y="9.398" size="1.016" layer="21" font="vector" ratio="12" rot="R90">RJHSE-548x</text>
 </plain>
 <attributes>
@@
 <attribute name="NAME" x="15.51" y="8.636" size="1" layer="25" font="vector" ratio="12" rot="R90" align="bottom-center"/>
 </element>
-<element name="SJ1" library="LoganSmith-Connectors" package="SJ_2" value="" x="5.715" y="8.255" smashed="yes" rot="MR0">
-<attribute name="NAME" x="8.609" y="9.825" size="1" layer="26" font="vector" ratio="12" rot="MR270"/>
-<attribute name="VALUE" x="7.285" y="6.65" size="0.5" layer="28" font="vector" ratio="12" rot="MR0"/>
-</element>
-<element name="SJ2" library="LoganSmith-Connectors" package="SJ_2" value="" x="5.715" y="19.685" smashed="yes" rot="MR0">
-<attribute name="NAME" x="8.609" y="21.255" size="1" layer="26" font="vector" ratio="12" rot="MR270"/>
-<attribute name="VALUE" x="7.285" y="18.08" size="0.5" layer="28" font="vector" ratio="12" rot="MR0"/>
-</element>
-<element name="J2" library="LoganSmith-Connectors" package="1X06_SQ1" value="M06SQ1" x="1.524" y="25.4" smashed="yes">
-<attribute name="VALUE" x="0.254" y="27.305" size="1" layer="27" font="vector" ratio="12"/>
-</element>
-<element name="J3" library="LoganSmith-Connectors" package="1X06_SQ1" value="M06SQ1" x="1.524" y="2.54" smashed="yes">
-<attribute name="VALUE" x="0.254" y="4.445" size="1" layer="27" font="vector" ratio="12"/>
-</element>
-<element name="LOGO1" library="SparkFun-Aesthetics" package="OSHW-LOGO-M" value="OSHW-LOGOM" x="11.176" y="13.97" rot="MR270"/>
+<element name="SJ1" library="LoganSmith-Connectors" package="SJ_2" value="" x="5.715" y="8.382" smashed="yes" rot="MR0">
+<attribute name="NAME" x="8.609" y="9.952" size="1" layer="26" font="vector" ratio="12" rot="MR270"/>
+<attribute name="VALUE" x="7.285" y="6.777" size="0.5" layer="28" font="vector" ratio="12" rot="MR0"/>
+</element>
+<element name="SJ2" library="LoganSmith-Connectors" package="SJ_2" value="" x="5.715" y="19.558" smashed="yes" rot="MR0">
+<attribute name="NAME" x="8.609" y="21.128" size="1" layer="26" font="vector" ratio="12" rot="MR270"/>
+<attribute name="VALUE" x="7.285" y="17.953" size="0.5" layer="28" font="vector" ratio="12" rot="MR0"/>
+</element>
+<element name="J2" library="LoganSmith-Connectors" package="1X06_SQ1" value="" x="1.778" y="25.4" smashed="yes">
+<attribute name="VALUE" x="0.508" y="27.305" size="1" layer="27" font="vector" ratio="12"/>
+</element>
+<element name="J3" library="LoganSmith-Connectors" package="1X06_SQ1" value="" x="1.778" y="2.54" smashed="yes">
+<attribute name="VALUE" x="0.508" y="4.445" size="1" layer="27" font="vector" ratio="12"/>
+</element>
+<element name="LOGO1" library="SparkFun-Aesthetics" package="OSHW-LOGO-M" value="OSHW-LOGOM" x="10.922" y="13.97" rot="MR90"/>
 </elements>
 <signals>
@@
 <contactref element="J1" pad="4"/>
 <contactref element="J3" pad="4"/>
-<wire x1="7.112" y1="13.462" x2="9.144" y2="11.43" width="0.254" layer="1"/>
-<wire x1="9.144" y1="11.43" x2="9.144" y2="2.54" width="0.254" layer="1"/>
+<wire x1="7.112" y1="13.462" x2="9.398" y2="11.176" width="0.254" layer="1"/>
+<wire x1="9.398" y1="11.176" x2="9.398" y2="2.54" width="0.254" layer="1"/>
 </signal>
 <signal name="N$6">
 <contactref element="J1" pad="3"/>
 <contactref element="J3" pad="3"/>
-<wire x1="6.604" y1="2.54" x2="6.604" y2="3.81" width="0.254" layer="16"/>
-<wire x1="6.604" y1="3.81" x2="8.636" y2="5.842" width="0.254" layer="16"/>
+<wire x1="6.858" y1="2.54" x2="6.858" y2="4.064" width="0.254" layer="16"/>
+<wire x1="6.858" y1="4.064" x2="8.636" y2="5.842" width="0.254" layer="16"/>
 <wire x1="8.636" y1="5.842" x2="8.636" y2="11.684" width="0.254" layer="16"/>
 <wire x1="8.636" y1="11.684" x2="7.874" y2="12.446" width="0.254" layer="16"/>
@@
 <contactref element="J1" pad="2"/>
 <contactref element="J3" pad="2"/>
-<wire x1="4.064" y1="2.54" x2="5.588" y2="4.064" width="0.254" layer="1"/>
-<wire x1="5.588" y1="4.064" x2="6.858" y2="4.064" width="0.254" layer="1"/>
+<wire x1="4.318" y1="2.54" x2="5.842" y2="4.064" width="0.254" layer="1"/>
+<wire x1="5.842" y1="4.064" x2="6.858" y2="4.064" width="0.254" layer="1"/>
 <wire x1="6.858" y1="4.064" x2="8.636" y2="5.842" width="0.254" layer="1"/>
 <wire x1="8.636" y1="5.842" x2="8.636" y2="9.906" width="0.254" layer="1"/>
@@
 <contactref element="J1" pad="1"/>
 <contactref element="J3" pad="1"/>
-<wire x1="1.524" y1="2.54" x2="1.524" y2="5.588" width="0.254" layer="1"/>
-<wire x1="1.524" y1="5.588" x2="0.508" y2="6.604" width="0.254" layer="1"/>
+<wire x1="1.778" y1="2.54" x2="1.778" y2="5.334" width="0.254" layer="1"/>
+<wire x1="1.778" y1="5.334" x2="0.508" y2="6.604" width="0.254" layer="1"/>
 <wire x1="0.508" y1="6.604" x2="0.508" y2="8.636" width="0.254" layer="1"/>
 <wire x1="0.508" y1="8.636" x2="2.286" y2="10.414" width="0.254" layer="1"/>
@@
 <wire x1="14.986" y1="15.56" x2="14.986" y2="13.97" width="0.254" layer="1"/>
 <wire x1="14.986" y1="12.38" x2="14.986" y2="13.97" width="0.254" layer="1"/>
-<wire x1="14.224" y1="25.4" x2="14.224" y2="20.574" width="0.254" layer="16"/>
-<wire x1="14.224" y1="20.574" x2="14.986" y2="19.812" width="0.254" layer="16"/>
+<wire x1="14.478" y1="25.4" x2="14.478" y2="20.32" width="0.254" layer="16"/>
+<wire x1="14.478" y1="20.32" x2="14.986" y2="19.812" width="0.254" layer="16"/>
 <wire x1="14.986" y1="19.812" x2="14.986" y2="13.97" width="0.254" layer="16"/>
 </signal>
@@
 <contactref element="J1" pad="LED2-"/>
 <contactref element="J3" pad="5"/>
-<wire x1="11.684" y1="2.54" x2="11.684" y2="5.334" width="0.254" layer="1"/>
-<wire x1="11.684" y1="5.334" x2="10.668" y2="6.35" width="0.254" layer="1"/>
+<wire x1="11.938" y1="2.54" x2="11.938" y2="5.08" width="0.254" layer="1"/>
+<wire x1="11.938" y1="5.08" x2="10.668" y2="6.35" width="0.254" layer="1"/>
 <wire x1="10.668" y1="6.35" x2="10.668" y2="17.272" width="0.254" layer="1"/>
 <wire x1="10.668" y1="17.272" x2="11.938" y2="18.542" width="0.254" layer="1"/>
@@
 <contactref element="J3" pad="6"/>
 <wire x1="11.938" y1="7.112" x2="13.208" y2="7.112" width="0.254" layer="1"/>
-<wire x1="13.208" y1="7.112" x2="14.224" y2="6.096" width="0.254" layer="1"/>
-<wire x1="14.224" y1="6.096" x2="14.224" y2="2.54" width="0.254" layer="1"/>
+<wire x1="13.208" y1="7.112" x2="14.478" y2="5.842" width="0.254" layer="1"/>
+<wire x1="14.478" y1="5.842" x2="14.478" y2="2.54" width="0.254" layer="1"/>
 </signal>
 <signal name="GND">
@@
 <contactref element="SJ1" pad="1"/>
 <contactref element="J1" pad="SHIELD@0"/>
-<wire x1="6.604" y1="8.255" x2="6.604" y2="6.223" width="0.508" layer="16"/>
+<wire x1="6.604" y1="8.382" x2="6.604" y2="6.223" width="0.508" layer="16"/>
 <wire x1="6.604" y1="6.223" x2="6.223" y2="5.842" width="0.508" layer="16"/>
 </signal>
@@
 <contactref element="J1" pad="SHEILD@1"/>
 <contactref element="SJ2" pad="1"/>
-<wire x1="6.604" y1="19.685" x2="6.604" y2="21.717" width="0.508" layer="16"/>
+<wire x1="6.604" y1="19.558" x2="6.604" y2="21.717" width="0.508" layer="16"/>
 <wire x1="6.604" y1="21.717" x2="6.223" y2="22.098" width="0.508" layer="16"/>
 </signal>
@@
 <contactref element="J2" pad="1"/>
 <contactref element="J1" pad="5"/>
-<wire x1="1.524" y1="25.4" x2="1.524" y2="22.352" width="0.254" layer="1"/>
-<wire x1="1.524" y1="22.352" x2="0.508" y2="21.336" width="0.254" layer="1"/>
+<wire x1="1.778" y1="25.4" x2="1.778" y2="22.606" width="0.254" layer="1"/>
+<wire x1="1.778" y1="22.606" x2="0.508" y2="21.336" width="0.254" layer="1"/>
 <wire x1="0.508" y1="21.336" x2="0.508" y2="16.256" width="0.254" layer="1"/>
 <wire x1="0.508" y1="16.256" x2="2.286" y2="14.478" width="0.254" layer="1"/>
@@
 <wire x1="8.636" y1="17.272" x2="8.636" y2="22.098" width="0.254" layer="16"/>
 <wire x1="8.636" y1="22.098" x2="6.858" y2="23.876" width="0.254" layer="16"/>
-<wire x1="6.858" y1="23.876" x2="5.588" y2="23.876" width="0.254" layer="16"/>
-<wire x1="5.588" y1="23.876" x2="4.064" y2="25.4" width="0.254" layer="16"/>
+<wire x1="6.858" y1="23.876" x2="5.842" y2="23.876" width="0.254" layer="16"/>
+<wire x1="5.842" y1="23.876" x2="4.318" y2="25.4" width="0.254" layer="16"/>
 </signal>
 <signal name="N$3">
@@
 <wire x1="5.334" y1="16.51" x2="5.334" y2="17.526" width="0.254" layer="1"/>
 <wire x1="5.334" y1="17.526" x2="8.636" y2="20.828" width="0.254" layer="1"/>
-<wire x1="8.636" y1="20.828" x2="8.636" y2="23.368" width="0.254" layer="1"/>
-<wire x1="8.636" y1="23.368" x2="6.604" y2="25.4" width="0.254" layer="1"/>
+<wire x1="8.636" y1="20.828" x2="8.636" y2="23.622" width="0.254" layer="1"/>
+<wire x1="8.636" y1="23.622" x2="6.858" y2="25.4" width="0.254" layer="1"/>
 </signal>
 <signal name="N$4">
 <contactref element="J2" pad="4"/>
 <contactref element="J1" pad="8"/>
-<wire x1="7.112" y1="17.526" x2="9.144" y2="19.558" width="0.254" layer="1"/>
-<wire x1="9.144" y1="19.558" x2="9.144" y2="25.4" width="0.254" layer="1"/>
+<wire x1="7.112" y1="17.526" x2="9.398" y2="19.812" width="0.254" layer="1"/>
+<wire x1="9.398" y1="19.812" x2="9.398" y2="25.4" width="0.254" layer="1"/>
 </signal>
 </signals>
